File: schematics/prototype/prototype.kicad_sch (KiCad schematic)
At the start: 0 parts

Commit message: feat(vasilis): added MCU side connections for FMC display
Also edited .gitignore for KiCad files
Parts:
- added U1: NUCLEO144-H743ZI-Q, Module:ST_Morpho_Connector_144_STLink, symbol MCU_Module:NUCLEO144-H743ZI
Connections:
- new net +3V3: U1.16 (+3V3)
- new net +5V: U1.18 (+5V)
- new net FMC_A16: U1.117 (PD11)
- new net FMC_D0: U1.118 (PD14)
- new net FMC_D1: U1.120 (PD15)
- new net FMC_D2: U1.57 (PD0)
- new net FMC_D3: U1.55 (PD1)
- new net FMC_D4: U1.116 (PE7)
- new net FMC_D5: U1.112 (PE8)
- new net FMC_D6: U1.124 (PE9)
- new net FMC_D7: U1.119 (PE10)
- new net FMC_NE1: U1.91 (PC7)
- new net FMC_NOE: U1.39 (PD4)
- new net FMC_NWE: U1.41 (PD5)
- new net GND: U1.111 (GND), U1.126 (GND), U1.135 (GND), U1.143 (GND), U1.144 (GND), U1.19 (GND), U1.20 (GND), U1.22 (GND), U1.49 (GND), U1.60 (GND), U1.71 (GND), U1.72 (GND), U1.8 (GND), U1.81 (GND), U1.92 (GND)
- new net LCD_BL_PWM: U1.87 (ETH_CRS_DV/PA7)
- new net LCD_RST: U1.43 (PD6)
- new net LCD_TE: U1.40 (PD3)
- no-connect marks 0 -> 109
Other:
- company: (none) -> Orsuka Industries
- title: (none) -> Kibble Prototype
